Commit message: REMOVE the collision box from my 3d (asus) camera, because it stuck out from the clean circle of the robot, causing odd path issues in DWA. My camera is within the circle, so it doesn't need its own collision box.

File: src/arlobot/arlobot_description/urdf/asus_xtion_pro_chrisl8.urdf.xacro (robot description, xacro)
@@ -39,5 +39,5 @@
         <origin xyz="0.0 0.0 0.0" rpy="0 0 0" />
         <geometry>
-        <box size="0.0730 0.2760 0.0720"/>
+        <box size="0.0 0.0 0.0"/>
       </geometry>
       </collision>
