Commit message: Move Asus Xtion xacro into my code so that RVIZ can find it on on systems without turtlebot debs installed.

File: src/arlobot/arlobot_description/urdf/asus_xtion_pro.urdf.xacro (robot description, xacro)
@@ -46,5 +46,5 @@
         <origin xyz="-0.01 0 0" rpy="${-M_PI/2} -${M_PI} ${-M_PI/2}"/>
         <geometry>
-          <mesh filename="package://turtlebot_description/meshes/sensors/asus_xtion_pro_live.dae" scale="${M_SCALE} ${M_SCALE} ${M_SCALE}"/>
+          <mesh filename="package://arlobot_description/meshes/sensors/asus_xtion_pro_live.dae" scale="${M_SCALE} ${M_SCALE} ${M_SCALE}"/>
         </geometry>
       </visual>

Commit message: Move missing files from turtlebot_descriptionn to arlobot_description.

File: src/arlobot/arlobot_description/urdf/asus_xtion_pro.urdf.xacro (robot description, xacro)
@@ -1,5 +1,5 @@
 <?xml version="1.0"?>
 <robot name="sensor_asus_xtion_pro" xmlns:xacro="http://ros.org/wiki/xacro">
-  <xacro:include filename="$(find turtlebot_description)/urdf/turtlebot_gazebo.urdf.xacro"/>
+  <xacro:include filename="$(find arlobot_description)/urdf/turtlebot_gazebo.urdf.xacro"/>
   <xacro:include filename="$(find arlobot_description)/urdf/turtlebot_properties.urdf.xacro"/>
   <!-- Xacro properties -->
@@ -33,5 +33,5 @@
         <origin xyz="-0.015 0.0035 0.004" rpy="0 0 0"/>
         <geometry>
-          <mesh filename="package://turtlebot_description/meshes/sensors/xtion_pro_camera.dae"/>
+          <mesh filename="package://arlobot_description/meshes/sensors/xtion_pro_camera.dae"/>
         </geometry>
       </visual>
@@ -74,5 +74,5 @@
         <origin xyz="0 0 0" rpy="${-M_PI/2} 0 0"/>
         <geometry>
-          <mesh filename="package://turtlebot_description/meshes/sensors/xtion_pro_stack.dae"/>
+          <mesh filename="package://arlobot_description/meshes/sensors/xtion_pro_stack.dae"/>
         </geometry>
       </visual>

File: src/arlobot/arlobot_description/urdf/asus_xtion_pro_chrisl8.urdf.xacro (robot description, xacro)
@@ -1,5 +1,5 @@
 <?xml version="1.0"?>
 <robot name="sensor_asus_xtion_pro" xmlns:xacro="http://ros.org/wiki/xacro">
-  <xacro:include filename="$(find turtlebot_description)/urdf/turtlebot_gazebo.urdf.xacro"/>
+  <xacro:include filename="$(find arlobot_description)/urdf/turtlebot_gazebo.urdf.xacro"/>
   <xacro:include filename="$(find arlobot_description)/urdf/turtlebot_properties_chrisl8.urdf.xacro"/>
   <!-- Xacro properties -->
@@ -33,5 +33,5 @@
         <origin xyz="-0.015 0.0035 0.004" rpy="0 0 0"/>
         <geometry>
-          <mesh filename="package://turtlebot_description/meshes/sensors/xtion_pro_camera.dae"/>
+          <mesh filename="package://arlobot_description/meshes/sensors/xtion_pro_camera.dae"/>
         </geometry>
       </visual>
@@ -74,5 +74,5 @@
         <origin xyz="0 0 0" rpy="${-M_PI/2} 0 0"/>
         <geometry>
-          <mesh filename="package://turtlebot_description/meshes/sensors/xtion_pro_stack.dae"/>
+          <mesh filename="package://arlobot_description/meshes/sensors/xtion_pro_stack.dae"/>
         </geometry>
       </visual>

Commit message: Fix scale on ASUS Xtion camera mesh for RVIZ

File: src/arlobot/arlobot_description/urdf/asus_xtion_pro.urdf.xacro (robot description, xacro)
@@ -33,5 +33,5 @@
         <origin xyz="-0.015 0.0035 0.004" rpy="0 0 0"/>
         <geometry>
-          <mesh filename="package://arlobot_description/meshes/sensors/xtion_pro_camera.dae"/>
+          <mesh filename="package://arlobot_description/meshes/sensors/xtion_pro_camera.dae" scale="0.001 0.001 0.001"/>
         </geometry>
       </visual>

File: src/arlobot/arlobot_description/urdf/asus_xtion_pro_chrisl8.urdf.xacro (robot description, xacro)
@@ -34,5 +34,5 @@
         <origin xyz="-0.015 0.0035 0.004" rpy="0 0 0"/>
         <geometry>
-          <mesh filename="package://arlobot_description/meshes/sensors/xtion_pro_camera.dae"/>
+          <mesh filename="package://arlobot_description/meshes/sensors/xtion_pro_camera.dae" scale="0.001 0.001 0.001"/>
         </geometry>
       </visual>
