Commit message: Cleanup description files and remove old turtlebot references.

File: src/arlobot/arlobot_description/urdf/3d_camera_position_chrisl8.urdf.xacro (robot description, xacro)
@@ -1,27 +1,11 @@
 <?xml version="1.0"?>
+  <!-- This file defines the 3D camera location.-->
+  <!-- See Readme.MD for hints on calibrating this -->
 <robot xmlns:xacro="http://ros.org/wiki/xacro">
-  <!--
-    These properties must be observed by any machine
-    that wants to be defined as a turtlebot. Refer
-    to the REP for more details.
-    http://www.ros.org/reps/rep-0119.html
-   -->
-  <!--
-   ======================================================================
-   - REP 119 : Rgb camera link relative to the Base link
-   ======================================================================
-     Base link is currently defined as the rotational centre on the bottom
-     of the base mould. For both create and kobuki this is actually exactly
-     the same 3d world point.
-     This may cause an issue with a base with much different floor clearance.
-     Should we be using base_footprint for this specification instead?
-     Note: REP needs to be updated with the information below
-     (currently in development and awaiting feedback)
-   -->
    <!-- This is how far forward or backward on the robot the camera is set. -->
 	<!-- Test this by setting the robot's axles exactly 1 meter from a wall, start up RVIZ with the robot at 0,0,0 on the grid, -->
 	<!-- and see if the wall lines up with the first 1 meter grid line from the robot. -->
 	<xacro:property name="cam_px" value="0.125" />
-<!--	<xacro:property name="cam_py" value="-0.0125" /> Y varies for different configurations. This is set in sensors_urdf -->
+	<!-- NOTE: cam_py, that is the Y offset, varies for different configurations. This is set in sensors_urdf instead of here -->
     <!-- This is the height of the camera. It isn't as essential as most settings, because we are using a "2D" map. -->
     <!-- However, setting it accurately can help with some use cases. -->

File: src/arlobot/arlobot_description/urdf/arlo.urdf.xacro (robot description, xacro)
@@ -4,5 +4,5 @@
   <xacro:property name="base_x" value="0.33" />
   <xacro:property name="base_y" value="0.33" />
-  <xacro:macro name="create">
+  <xacro:macro name="arlobot">
     <material name="Green">
       <color rgba="0.0 0.8 0.0 1.0"/>
@@ -282,6 +282,6 @@
   <!-- XV11 Neato Laser scanner. Hopefully it is exactly in the center. :) -->
   <joint name="neato_laser_joint" type="fixed">
-    <!-- Minor adjustments based on ligning up XV11 output with 3D Sensor output -->
-    <!-- So if the 3D sensor is misallgined the XV11 is off by the same amount -->
+    <!-- Minor adjustments based on lining up XV11 output with 3D Sensor output -->
+    <!-- So if the 3D sensor is misaligned the XV11 is off by the same amount -->
     <origin xyz="0.015 -0.02 0.11875" rpy="-0.025 0 0" />
     <parent link="base_link" />
@@ -303,5 +303,5 @@
   </link>
   </xacro:macro>
-  <xacro:macro name="turtlebot_standoff_5in" params="parent number x_loc y_loc z_loc">
+  <xacro:macro name="arlobot_standoff_5in" params="parent number x_loc y_loc z_loc">
     <joint name="standoff_5in_${number}_joint" type="fixed">
       <origin xyz="${x_loc} ${y_loc} ${z_loc}" rpy="0 0 0" />
@@ -364,8 +364,8 @@
       </collision>
     </link>
-    <turtlebot_standoff_5in parent="${parent}" number="0" x_loc="0.0676402" y_loc="0.1314196" z_loc="0.06825"/>
-    <turtlebot_standoff_5in parent="${parent}" number="1" x_loc="0.0676402" y_loc="-0.1314196" z_loc="0.06825"/>
-    <turtlebot_standoff_5in parent="${parent}" number="2" x_loc="-0.052832" y_loc="-0.1314196" z_loc="0.06825"/>
-    <turtlebot_standoff_5in parent="${parent}" number="3" x_loc="-0.052832" y_loc="0.1314196" z_loc="0.06825"/>
+    <arlobot_standoff_5in parent="${parent}" number="0" x_loc="0.0676402" y_loc="0.1314196" z_loc="0.06825"/>
+    <arlobot_standoff_5in parent="${parent}" number="1" x_loc="0.0676402" y_loc="-0.1314196" z_loc="0.06825"/>
+    <arlobot_standoff_5in parent="${parent}" number="2" x_loc="-0.052832" y_loc="-0.1314196" z_loc="0.06825"/>
+    <arlobot_standoff_5in parent="${parent}" number="3" x_loc="-0.052832" y_loc="0.1314196" z_loc="0.06825"/>
   </xacro:macro>
 </robot>

File: src/arlobot/arlobot_description/urdf/arlo_2stack.urdf.xacro (robot description, xacro)
@@ -4,5 +4,5 @@
   <xacro:property name="base_x" value="0.33" />
   <xacro:property name="base_y" value="0.33" />
-  <xacro:macro name="create">
+  <xacro:macro name="arlobot">
     <material name="Green">
       <color rgba="0.0 0.8 0.0 1.0"/>
@@ -280,30 +280,8 @@
       </inertial>
     </link>
-  <!-- XV11 Neato Laser scanner. Hopefully it is exactly in the center. :) -->
-  <!--   <joint name="neato_laser_joint" type="fixed"> -->
-       <!-- Minor adjustments based on lining up XV11 output with 3D Sensor output -->
-       <!-- So if the 3D sensor is misaligned the XV11 is off by the same amount -->
-  <!--     <origin xyz="0.015 -0.02 0.11875" rpy="-0.025 0 0" /> -->
-  <!--     <parent link="base_link" /> -->
-  <!--     <child link="neato_laser" /> -->
-  <!--   </joint> -->
-  <!--   <link name="neato_laser"> -->
-  <!--     <visual> -->
-  <!--       <geometry> -->
-  <!--         <box size="0.0 0.0 0.0" /> -->
-  <!--       </geometry> -->
-  <!--     </visual> -->
-  <!--     <inertial> -->
-  <!--       <mass value="0.001" /> -->
-  <!--       <origin xyz="0 0 0" /> -->
-  <!--       <inertia ixx="0.0001" ixy="0.0" ixz="0.0" -->
-  <!--         iyy="0.0001" iyz="0.0" -->
-  <!--         izz="0.0001" /> -->
-  <!--     </inertial> -->
-  <!--   </link> -->
   <!-- Scanse Sweep Sensor on top of robot -->
      <joint name="scanse_sweep_joint" type="fixed">
-        Minor adjustments based on lining up Scanse Sweep output with 3D Sensor output
-        So if the 3D sensor is misaligned the Scanse Sweep is off by the same amount
+       <!-- Minor adjustments based on lining up Scanse Sweep output with 3D Sensor output -->
+       <!-- So if the 3D sensor is misaligned the Scanse Sweep is off by the same amount -->
        <origin xyz="0.15 0.0 0.269107" rpy="0 0 3.13" />
        <parent link="base_link" />
@@ -325,5 +303,5 @@
      </link>
      </xacro:macro>
-  <xacro:macro name="turtlebot_standoff_5in" params="parent number x_loc y_loc z_loc">
+  <xacro:macro name="arlobot_standoff_5in" params="parent number x_loc y_loc z_loc">
     <joint name="standoff_5in_${number}_joint" type="fixed">
       <origin xyz="${x_loc} ${y_loc} ${z_loc}" rpy="0 0 0" />
@@ -386,8 +364,8 @@
       </collision>
     </link>
-    <turtlebot_standoff_5in parent="${parent}" number="0" x_loc="0.0676402" y_loc="0.1314196" z_loc="0.06825"/>
-    <turtlebot_standoff_5in parent="${parent}" number="1" x_loc="0.0676402" y_loc="-0.1314196" z_loc="0.06825"/>
-    <turtlebot_standoff_5in parent="${parent}" number="2" x_loc="-0.052832" y_loc="-0.1314196" z_loc="0.06825"/>
-    <turtlebot_standoff_5in parent="${parent}" number="3" x_loc="-0.052832" y_loc="0.1314196" z_loc="0.06825"/>
+    <arlobot_standoff_5in parent="${parent}" number="0" x_loc="0.0676402" y_loc="0.1314196" z_loc="0.06825"/>
+    <arlobot_standoff_5in parent="${parent}" number="1" x_loc="0.0676402" y_loc="-0.1314196" z_loc="0.06825"/>
+    <arlobot_standoff_5in parent="${parent}" number="2" x_loc="-0.052832" y_loc="-0.1314196" z_loc="0.06825"/>
+    <arlobot_standoff_5in parent="${parent}" number="3" x_loc="-0.052832" y_loc="0.1314196" z_loc="0.06825"/>
     <joint name="plate_1_joint" type="fixed">
       <origin xyz="0 0 0.1365" rpy="0 0 0" />
@@ -419,8 +397,8 @@
       </collision>
     </link>
-    <turtlebot_standoff_5in parent="plate_0_link" number="4" x_loc="0.0676402" y_loc="0.1314196" z_loc="0.06825"/>
-    <turtlebot_standoff_5in parent="plate_0_link" number="5" x_loc="0.0676402" y_loc="-0.1314196" z_loc="0.06825"/>
-    <turtlebot_standoff_5in parent="plate_0_link" number="6" x_loc="-0.052832" y_loc="-0.1314196" z_loc="0.06825"/>
-    <turtlebot_standoff_5in parent="plate_0_link" number="7" x_loc="-0.052832" y_loc="0.1314196" z_loc="0.06825"/>
+    <arlobot_standoff_5in parent="plate_0_link" number="4" x_loc="0.0676402" y_loc="0.1314196" z_loc="0.06825"/>
+    <arlobot_standoff_5in parent="plate_0_link" number="5" x_loc="0.0676402" y_loc="-0.1314196" z_loc="0.06825"/>
+    <arlobot_standoff_5in parent="plate_0_link" number="6" x_loc="-0.052832" y_loc="-0.1314196" z_loc="0.06825"/>
+    <arlobot_standoff_5in parent="plate_0_link" number="7" x_loc="-0.052832" y_loc="0.1314196" z_loc="0.06825"/>
   </xacro:macro>
 </robot>

File: src/arlobot/arlobot_description/urdf/asus_xtion_pro.urdf.xacro (robot description, xacro)
@@ -1,6 +1,5 @@
 <?xml version="1.0"?>
 <robot name="sensor_asus_xtion_pro" xmlns:xacro="http://ros.org/wiki/xacro">
-  <xacro:include filename="$(find arlobot_description)/urdf/turtlebot_gazebo.urdf.xacro"/>
-  <xacro:include filename="$(find arlobot_description)/urdf/turtlebot_properties.urdf.xacro"/>
+  <xacro:include filename="$(find arlobot_description)/urdf/3d_camera_position.urdf.xacro"/>
   <!-- Xacro properties -->
   <xacro:property name="M_SCALE" value="0.001"/>
@@ -8,5 +7,5 @@
   <xacro:property name="asus_xtion_pro_depth_rel_rgb_py" value="0.0270" />
   <xacro:property name="asus_xtion_pro_cam_rel_rgb_py"   value="-0.0220" />
-  <!-- Parameterised in part by the values in turtlebot_properties.urdf.xacro -->
+  <!-- Parameterised in part by the values in 3d_camera_position.urdf.xacro -->
   <xacro:macro name="sensor_asus_xtion_pro" params="parent">
     <joint name="camera_rgb_joint" type="fixed">
@@ -62,6 +61,4 @@
     </joint>
     <link name="camera_depth_optical_frame"/>
-    <!-- RGBD sensor for simulation, same as Kinect -->
-    <turtlebot_sim_3dsensor/>
     <!-- Asus mount -->
     <joint name="mount_asus_xtion_pro_joint" type="fixed">

File: src/arlobot/arlobot_description/urdf/asus_xtion_pro_chrisl8.urdf.xacro (robot description, xacro)
@@ -1,6 +1,5 @@
 <?xml version="1.0"?>
 <robot name="sensor_asus_xtion_pro" xmlns:xacro="http://ros.org/wiki/xacro">
-  <xacro:include filename="$(find arlobot_description)/urdf/turtlebot_gazebo.urdf.xacro"/>
-  <xacro:include filename="$(find arlobot_description)/urdf/turtlebot_properties_chrisl8.urdf.xacro"/>
+  <xacro:include filename="$(find arlobot_description)/urdf/3d_camera_position_chrisl8.urdf.xacro"/>
   <!-- Xacro properties -->
   <xacro:property name="M_SCALE" value="0.001"/>
@@ -9,5 +8,5 @@
   <!-- Camera left/right offset. Camera is actually off center in the unit, so -0.0220 makes it physically centered. -->
   <xacro:property name="asus_xtion_pro_cam_rel_rgb_py"   value="-0.0220" />
-  <!-- Parameterised in part by the values in turtlebot_properties.urdf.xacro -->
+  <!-- Parameterised in part by the values in 3d_camera_position_chrisl8.urdf.xacro -->
   <xacro:macro name="sensor_asus_xtion_pro" params="parent">
     <joint name="camera_rgb_joint" type="fixed">
@@ -63,6 +62,4 @@
     </joint>
     <link name="camera_depth_optical_frame"/>
-    <!-- RGBD sensor for simulation, same as Kinect -->
-    <turtlebot_sim_3dsensor/>
   </xacro:macro>
 </robot>

File: src/arlobot/arlobot_description/urdf/common_chrisl8.urdf.xacro (robot description, xacro)
@@ -7,17 +7,11 @@
   <!-- It is required by asus_xtion_pro.urdf.xacro -->
   <xacro:property name="M_PI" value="3.1415926535897931" />
-  <!--
-    These properties must be observed by any machine
-    that wants to be defined as a turtlebot. Refer
-    to the REP for more details.
-    http://www.ros.org/reps/rep-0119.html
-   -->
-  <!-- This is where the Xtion location is set. I do not think it has any other function. -->
-  <xacro:include filename="$(find arlobot_description)/urdf/turtlebot_properties_chrisl8.urdf.xacro"/>
+  <!-- This is where the 3D camera location is set. -->
+  <xacro:include filename="$(find arlobot_description)/urdf/3d_camera_position_chrisl8.urdf.xacro"/>
   <!-- ArloBot -->
   <xacro:include filename="$(find arlobot_description)/urdf/arlo_2stack.urdf.xacro"/>
   <!-- 3D Sensor -->
   <xacro:include filename="$(find arlobot_description)/urdf/asus_xtion_pro_chrisl8.urdf.xacro"/>
-  <create/>
+  <arlobot/>
   <stack_circles parent="base_link"/>
   <sensor_asus_xtion_pro  parent="base_link"/>

File: src/arlobot/arlobot_description/urdf/common_default.urdf.xacro (robot description, xacro)
@@ -7,18 +7,11 @@
   <!-- It is required by asus_xtion_pro.urdf.xacro -->
   <xacro:property name="M_PI" value="3.1415926535897931" />
-  <!--
-    These properties must be observed by any machine
-    that wants to be defined as a turtlebot. Refer
-    to the REP for more details.
-    http://www.ros.org/reps/rep-0119.html
-   -->
-  <!-- This is where the Xtion location is set. I do not think it has any other function. -->
-  <xacro:include filename="$(find arlobot_description)/urdf/turtlebot_properties.urdf.xacro"/>
+  <!-- This is where the 3D camera location is set. -->
+  <xacro:include filename="$(find arlobot_description)/urdf/3d_camera_position.urdf.xacro"/>
   <!-- ArloBot -->
-  <!-- There is no actual ArloBot model, I never made one. -->
   <xacro:include filename="$(find arlobot_description)/urdf/arlo.urdf.xacro"/>
   <!-- 3D Sensor -->
   <xacro:include filename="$(find arlobot_description)/urdf/asus_xtion_pro.urdf.xacro"/>
-  <create/>
+  <arlobot/>
   <stack_circles parent="base_link"/>
   <sensor_asus_xtion_pro  parent="base_link"/>
