Commit message: Prepare for Kinetic Kame release
Use the environment variable in place of 'indigo' for ROS Distro.
Update xacro description files to be standards compliant.

File: src/arlobot/arlobot_description/urdf/arlo_2stack.urdf.xacro (robot description, xacro)
@@ -2,6 +2,6 @@
 <robot name="arlobot_hardware" xmlns:xacro="http://ros.org/wiki/xacro">
   <!-- Macro for ArloBot body. -->
-  <property name="base_x" value="0.33" />
-  <property name="base_y" value="0.33" />
+  <xacro:property name="base_x" value="0.33" />
+  <xacro:property name="base_y" value="0.33" />
   <xacro:macro name="create">
     <material name="Green">

File: src/arlobot/arlobot_description/urdf/turtlebot_properties.urdf.xacro (robot description, xacro)
@@ -1,4 +1,4 @@
 <?xml version="1.0"?>
-<robot>
+<robot xmlns:xacro="http://ros.org/wiki/xacro">
   <!--
     These properties must be observed by any machine
@@ -19,9 +19,9 @@
      (currently in development and awaiting feedback)
    -->
-	<property name="cam_px" value="-0.17745" />
-	<property name="cam_py" value="0.027" />
-	<property name="cam_pz" value="0.2985" />
-	<property name="cam_or" value="-0.01" />
-	<property name="cam_op" value="0" />
-	<property name="cam_oy" value="0" />
+	<xacro:property name="cam_px" value="-0.17745" />
+	<xacro:property name="cam_py" value="0.027" />
+	<xacro:property name="cam_pz" value="0.2985" />
+	<xacro:property name="cam_or" value="-0.01" />
+	<xacro:property name="cam_op" value="0" />
+	<xacro:property name="cam_oy" value="0" />
 </robot>

File: src/arlobot/arlobot_description/urdf/turtlebot_properties_chrisl8.urdf.xacro (robot description, xacro)
@@ -1,4 +1,4 @@
 <?xml version="1.0"?>
-<robot>
+<robot xmlns:xacro="http://ros.org/wiki/xacro">
   <!--
     These properties must be observed by any machine
@@ -19,9 +19,9 @@
      (currently in development and awaiting feedback)
    -->
-	<property name="cam_px" value="0.19" />
-<!--	<property name="cam_py" value="-0.0125" /> Y varies for different configurations. get sets in sensors_urdf -->
-	<property name="cam_pz" value="0.17" />
-	<property name="cam_or" value="0" />
-	<property name="cam_op" value="0" />
-	<property name="cam_oy" value="0" />
+	<xacro:property name="cam_px" value="0.19" />
+<!--	<xacro:property name="cam_py" value="-0.0125" /> Y varies for different configurations. get sets in sensors_urdf -->
+	<xacro:property name="cam_pz" value="0.17" />
+	<xacro:property name="cam_or" value="0" />
+	<xacro:property name="cam_op" value="0" />
+	<xacro:property name="cam_oy" value="0" />
 </robot>

Commit message: Add RPLIDAR to my description file.

File: src/arlobot/arlobot_description/urdf/arlo_2stack.urdf.xacro (robot description, xacro)
@@ -302,4 +302,27 @@
        </inertial>
      </link>
+  <!-- RPLIDAR on top of robot -->
+     <joint name="rplidar_joint" type="fixed">
+       <!-- Minor adjustments based on lining up Scanse Sweep output with 3D Sensor output -->
+       <!-- So if the 3D sensor is misaligned the Scanse Sweep is off by the same amount -->
+       <!-- NOTE: The "FRONT" of the RPLIDAR A2/3 is the point where the cord comes out. -->
+       <origin xyz="0.15 0.0 0.269107" rpy="0 0 3.13" />
+       <parent link="base_link" />
+       <child link="rplidar" />
+     </joint>
+     <link name="rplidar">
+       <visual>
+         <geometry>
+           <box size="0.0 0.0 0.0" />
+         </geometry>
+       </visual>
+       <inertial>
+         <mass value="0.001" />
+         <origin xyz="0 0 0" />
+         <inertia ixx="0.0001" ixy="0.0" ixz="0.0"
+           iyy="0.0001" iyz="0.0"
+           izz="0.0001" />
+       </inertial>
+     </link>
      </xacro:macro>
   <xacro:macro name="arlobot_standoff_5in" params="parent number x_loc y_loc z_loc">

Commit message: Tweak my RPLIDAR location in the description files.

File: src/arlobot/arlobot_description/urdf/arlo_2stack.urdf.xacro (robot description, xacro)
@@ -304,8 +304,13 @@
   <!-- RPLIDAR on top of robot -->
      <joint name="rplidar_joint" type="fixed">
-       <!-- Minor adjustments based on lining up Scanse Sweep output with 3D Sensor output -->
-       <!-- So if the 3D sensor is misaligned the Scanse Sweep is off by the same amount -->
+       <!-- WARNING: The 'rpy' means Roll, Pitch, Yaw, but in the static_transform_publisher the order -->
+       <!-- is Yaw, Pitch, Roll !!!  So don't forget to translate those! -->
+       <!-- The best way to tweak this is to delete this section, start the robot, and use -->
+       <!-- staticTransformExample.sh to broadcast this transform while watching in RVIZ, -->
+       <!-- and keep tweaking the numbers and killing and restarting that transform broadcaster. -->
        <!-- NOTE: The "FRONT" of the RPLIDAR A2/3 is the point where the cord comes out. -->
-       <origin xyz="0.15 0.0 0.269107" rpy="0 0 3.13" />
+       <!-- Hence the r of 3.1 to rotate it half way around.  -->
+       <!-- The height is set even with the top plate. It shouldn't matter really. -->
+       <origin xyz="0.125 0.0 0.269107" rpy="0.0 0.0 3.1" />
        <parent link="base_link" />
        <child link="rplidar" />
