Commit message: Turn my RPLIDAR around in attempt to fix issues with Slam Toolbox and map rotating randomly.

File: arlobot_ros/urdf/arlo_2stack.urdf.xacro (robot description, xacro)
@@ -315,5 +315,5 @@
       <!-- Hence the r of 3.1 to rotate it half way around.  -->
       <!-- The height is set even with the top plate. It shouldn't matter really. -->
-      <origin xyz="0.125 0.0 0.269107" rpy="0.0 0.0 3.1"/>
+      <origin xyz="0.125 0.0 0.269107" rpy="0.0 0.0 0.0"/>
       <parent link="base_link"/>
       <child link="rplidar"/>
