Commit message: Simplify caster mesh
 - Reduced  vertices from 44,232 to about 5,000
 - I'm not sure this even matters, but it has been on my todo list for ages.
 - The original is still in the repo if somebody wants it.

File: arlobot_ros/urdf/arlo.urdf.xacro (robot description, xacro)
@@ -92,5 +92,5 @@
         <origin xyz="0 0 0" rpy="-1.5707 0 1.5707"/>
         <geometry>
-          <mesh filename="package://arlobot_ros/meshes/28971-Caster-Wheel-Kit-v1.0.stl"/>
+          <mesh filename="package://arlobot_ros/meshes/28971-Caster-Wheel-Kit-v1.0_simplified.stl"/>
         </geometry>
         <material name="light_grey">
@@ -115,5 +115,5 @@
         <origin xyz="0 0 0" rpy="-1.5707 0 1.5707"/>
         <geometry>
-          <mesh filename="package://arlobot_ros/meshes/28971-Caster-Wheel-Kit-v1.0.stl"/>
+          <mesh filename="package://arlobot_ros/meshes/28971-Caster-Wheel-Kit-v1.0_simplified.stl"/>
         </geometry>
         <material name="light_grey">

File: arlobot_ros/urdf/arlo_2stack.urdf.xacro (robot description, xacro)
@@ -92,5 +92,5 @@
         <origin xyz="0 0 0" rpy="-1.5707 0 1.5707"/>
         <geometry>
-          <mesh filename="package://arlobot_ros/meshes/28971-Caster-Wheel-Kit-v1.0.stl"/>
+          <mesh filename="package://arlobot_ros/meshes/28971-Caster-Wheel-Kit-v1.0_simplified.stl"/>
         </geometry>
         <material name="light_grey">
@@ -115,5 +115,5 @@
         <origin xyz="0 0 0" rpy="-1.5707 0 1.5707"/>
         <geometry>
-          <mesh filename="package://arlobot_ros/meshes/28971-Caster-Wheel-Kit-v1.0.stl"/>
+          <mesh filename="package://arlobot_ros/meshes/28971-Caster-Wheel-Kit-v1.0_simplified.stl"/>
         </geometry>
         <material name="light_grey">
