Commit message: Clean up and fix URDF file source and generation.

File: arlobot_ros/urdf/3d_camera_position.urdf.xacro (robot description, xacro)
@@ -6,11 +6,11 @@
   <!-- Test this by setting the robot's axles exactly 1 meter from a wall, start up RVIZ with the robot at 0,0,0 on the grid, -->
   <!-- and see if the wall lines up with the first 1 meter grid line from the robot. -->
-  <xacro:property name="cam_px" value="-0.17745"/>
+  <xacro:property name="cam_px" value="0.125"/>
   <!-- NOTE: cam_py, that is the Y offset, varies for different configurations. This is set in sensors_urdf instead of here -->
   <!-- This is the height of the camera. It isn't as essential as most settings, because we are using a "2D" map. -->
   <!-- However, setting it accurately can help with some use cases. -->
-  <xacro:property name="cam_pz" value="0.2985"/>
+  <xacro:property name="cam_pz" value="0.17"/>
   <!-- This is the tilt across the horizontal when looking straight at the camera. Probably important, but hard to see if it is. -->
-  <xacro:property name="cam_or" value="-0.01"/>
+  <xacro:property name="cam_or" value="0"/>
   <!-- This is the tilt causing the camera to look "up" or "down". -->
   <xacro:property name="cam_op" value="0"/>
@@ -18,4 +18,4 @@
   <!-- Test this by setting the robot's axles exactly 1 meter from a wall, start up RVIZ with the robot at 0,0,0 on the grid, -->
   <!-- and see if the wall lines up straight with the grid line. -->
-  <xacro:property name="cam_oy" value="0"/>
+  <xacro:property name="cam_oy" value="-0.005"/>
 </robot>

File: arlobot_ros/urdf/arlo.urdf.xacro (robot description, xacro)
@@ -283,29 +283,9 @@
       </inertial>
     </link>
-    <!-- XV11 Neato Laser scanner. -->
-    <!--    NOTE: This is no longer used on my robot, only on my stationary test rig. -->
-    <joint name="neato_laser_joint" type="fixed">
-      <origin xyz="0.0 0.0 0.0" rpy="0.0 0 0"/>
-      <parent link="base_link"/>
-      <child link="neato_laser"/>
-    </joint>
-    <link name="neato_laser">
-      <visual>
-        <geometry>
-          <box size="0.1 0.1 0.1"/>
-        </geometry>
-      </visual>
-      <inertial>
-        <mass value="0.001"/>
-        <origin xyz="0 0 0"/>
-        <inertia ixx="0.0001" ixy="0.0" ixz="0.0"
-                 iyy="0.0001" iyz="0.0"
-                 izz="0.0001"/>
-      </inertial>
-    </link>
-    <!-- Scanse Sweep rotary scanner. -->
-    <!--    NOTE: This is no longer used on my robot, only on my stationary test rig. -->
+    <!-- Scanse Sweep Sensor on top of robot -->
     <joint name="scanse_sweep_joint" type="fixed">
-      <origin xyz="0.0 0.0 0.0" rpy="0.0 0 0"/>
+      <!-- Minor adjustments based on lining up Scanse Sweep output with 3D Sensor output -->
+      <!-- So if the 3D sensor is misaligned the Scanse Sweep is off by the same amount -->
+      <origin xyz="0.15 0.0 0.269107" rpy="0 0 3.13"/>
       <parent link="base_link"/>
       <child link="scanse_sweep"/>
@@ -314,5 +294,33 @@
       <visual>
         <geometry>
-          <box size="0.1 0.1 0.1"/>
+          <box size="0.0 0.0 0.0"/>
+        </geometry>
+      </visual>
+      <inertial>
+        <mass value="0.001"/>
+        <origin xyz="0 0 0"/>
+        <inertia ixx="0.0001" ixy="0.0" ixz="0.0"
+                 iyy="0.0001" iyz="0.0"
+                 izz="0.0001"/>
+      </inertial>
+    </link>
+    <!-- RPLIDAR on top of robot -->
+    <joint name="rplidar_joint" type="fixed">
+      <!-- WARNING: The 'rpy' means Roll, Pitch, Yaw, but in the static_transform_publisher the order -->
+      <!-- is Yaw, Pitch, Roll !!!  So don't forget to translate those! -->
+      <!-- The best way to tweak this is to delete this section, start the robot, and use -->
+      <!-- staticTransformExample.sh to broadcast this transform while watching in RVIZ, -->
+      <!-- and keep tweaking the numbers and killing and restarting that transform broadcaster. -->
+      <!-- NOTE: The "FRONT" of the RPLIDAR A2/3 is the point where the cord comes out. -->
+      <!-- Hence the r of 3.1 to rotate it half way around.  -->
+      <!-- The height is set even with the top plate. It shouldn't matter really. -->
+      <origin xyz="0.125 0.0 0.269107" rpy="0.0 0.0 0.0"/>
+      <parent link="base_link"/>
+      <child link="rplidar"/>
+    </joint>
+    <link name="rplidar">
+      <visual>
+        <geometry>
+          <box size="0.0 0.0 0.0"/>
         </geometry>
       </visual>
@@ -388,11 +396,48 @@
     </link>
     <xacro:arlobot_standoff_5in parent="${parent}" number="0" x_loc="0.0676402" y_loc="0.1314196"
-                                z_loc="0.06825"/>
+                          z_loc="0.06825"/>
     <xacro:arlobot_standoff_5in parent="${parent}" number="1" x_loc="0.0676402" y_loc="-0.1314196"
-                                z_loc="0.06825"/>
+                          z_loc="0.06825"/>
     <xacro:arlobot_standoff_5in parent="${parent}" number="2" x_loc="-0.052832" y_loc="-0.1314196"
-                                z_loc="0.06825"/>
+                          z_loc="0.06825"/>
     <xacro:arlobot_standoff_5in parent="${parent}" number="3" x_loc="-0.052832" y_loc="0.1314196"
-                                z_loc="0.06825"/>
+                          z_loc="0.06825"/>
+    <joint name="plate_1_joint" type="fixed">
+      <origin xyz="0 0 0.1365" rpy="0 0 0"/>
+      <parent link="plate_0_link"/>
+      <child link="plate_1_link"/>
+    </joint>
+    <link name="plate_1_link">
+      <inertial>
+        <mass value="0.01"/>
+        <origin xyz="0 0 0"/>
+        <inertia ixx="0.01" ixy="0.0" ixz="0.0"
+                 iyy="0.01" iyz="0.0"
+                 izz="0.01"/>
+      </inertial>
+      <visual>
+        <origin xyz=" 0 0 0 " rpy="0 0 0"/>
+        <geometry>
+          <cylinder length="0.0095" radius="0.2245"/>
+        </geometry>
+        <material name="veryDarkGrey">
+          <color rgba=".2 .2 .2 1"/>
+        </material>
+      </visual>
+      <collision>
+        <origin xyz="0.0 0.0 0.0" rpy="0 0 0"/>
+        <geometry>
+          <cylinder length="0.0095" radius="0.2245"/>
+        </geometry>
+      </collision>
+    </link>
+    <xacro:arlobot_standoff_5in parent="plate_0_link" number="4" x_loc="0.0676402" y_loc="0.1314196"
+                          z_loc="0.06825"/>
+    <xacro:arlobot_standoff_5in parent="plate_0_link" number="5" x_loc="0.0676402" y_loc="-0.1314196"
+                          z_loc="0.06825"/>
+    <xacro:arlobot_standoff_5in parent="plate_0_link" number="6" x_loc="-0.052832" y_loc="-0.1314196"
+                          z_loc="0.06825"/>
+    <xacro:arlobot_standoff_5in parent="plate_0_link" number="7" x_loc="-0.052832" y_loc="0.1314196"
+                          z_loc="0.06825"/>
   </xacro:macro>
 </robot>

File: arlobot_ros/urdf/asus_xtion_pro.urdf.xacro (robot description, xacro)
@@ -1,11 +1,12 @@
 <?xml version="1.0"?>
 <robot name="sensor_asus_xtion_pro" xmlns:xacro="http://ros.org/wiki/xacro">
-  <xacro:include filename="$(find arlobot_ros)/urdf/3d_camera_position.urdf.xacro"/>
+  <xacro:include filename="$(find arlobot_ros)/urdf/3d_camera_position_chrisl8.urdf.xacro"/>
   <!-- Xacro properties -->
   <xacro:property name="M_SCALE" value="0.001"/>
   <xacro:property name="asus_xtion_pro_cam_py" value="0.0205"/>
   <xacro:property name="asus_xtion_pro_depth_rel_rgb_py" value="0.0270"/>
+  <!-- Camera left/right offset. Camera is actually off center in the unit, so -0.0220 makes it physically centered. -->
   <xacro:property name="asus_xtion_pro_cam_rel_rgb_py" value="-0.0220"/>
-  <!-- Parameterised in part by the values in 3d_camera_position.urdf.xacro -->
+  <!-- Parameterised in part by the values in 3d_camera_position_chrisl8.urdf.xacro -->
   <xacro:macro name="sensor_asus_xtion_pro" params="parent">
     <joint name="camera_rgb_joint" type="fixed">
@@ -39,5 +40,5 @@
         <origin xyz="0.0 0.0 0.0" rpy="0 0 0"/>
         <geometry>
-          <box size="0.0730 0.2760 0.0720"/>
+          <box size="0.0 0.0 0.0"/>
         </geometry>
       </collision>
@@ -62,31 +63,4 @@
     </joint>
     <link name="camera_depth_optical_frame"/>
-    <!-- Asus mount -->
-    <joint name="mount_asus_xtion_pro_joint" type="fixed">
-      <origin xyz="-0.1024 0.0 0.272" rpy="0 0 0"/>
-      <parent link="${parent}"/>
-      <child link="mount_asus_xtion_pro_link"/>
-    </joint>
-    <link name="mount_asus_xtion_pro_link">
-      <visual>
-        <origin xyz="0 0 0" rpy="${-M_PI/2} 0 0"/>
-        <geometry>
-          <mesh filename="package://arlobot_ros/meshes/sensors/xtion_pro_stack.dae"/>
-        </geometry>
-      </visual>
-      <collision>
-        <origin xyz="0.0 0.0 0.0" rpy="0 0 0"/>
-        <geometry>
-          <box size="0.0330 0.2760 0.0120"/>
-        </geometry>
-      </collision>
-      <inertial>
-        <mass value="0.170"/>
-        <origin xyz="0 0 0"/>
-        <inertia ixx="0.001152600" ixy="0.0" ixz="0.0"
-                 iyy="0.000148934" iyz="0.0"
-                 izz="0.001154654"/>
-      </inertial>
-    </link>
   </xacro:macro>
 </robot>

File: arlobot_ros/urdf/common.urdf.xacro (robot description, xacro)
@@ -8,9 +8,10 @@
   <xacro:property name="M_PI" value="3.1415926535897931"/>
   <!-- This is where the 3D camera location is set. -->
-  <xacro:include filename="$(find arlobot_ros)/urdf/3d_camera_position_chrisl8.urdf.xacro"/>
+  <xacro:include filename="$(find arlobot_ros)/urdf/3d_camera_position.urdf.xacro"/>
   <!-- ArloBot -->
-  <xacro:include filename="$(find arlobot_ros)/urdf/arlo_2stack.urdf.xacro"/>
+  <xacro:include filename="$(find arlobot_ros)/urdf/arlo.urdf.xacro"/>
   <!-- 3D Sensor -->
-  <xacro:include filename="$(find arlobot_ros)/urdf/asus_xtion_pro_chrisl8.urdf.xacro"/>
+  <!-- TODO: Why is this still here? Can I safely remove it? -->
+  <xacro:include filename="$(find arlobot_ros)/urdf/asus_xtion_pro.urdf.xacro"/>
   <xacro:arlobot/>
   <xacro:stack_circles parent="base_link"/>
