Commit message: Refactor URDF model view and make one working rviz file.

File: urdf/arlo.urdf.xacro (robot description, xacro)
@@ -90,7 +90,7 @@
       </inertial>
       <visual>
-        <origin xyz="0 0 0" rpy="-1.5707 0 1.5707"/>
-        <geometry>
-          <mesh filename="package://arlobot_ros/meshes/28971-Caster-Wheel-Kit-v1.0_simplified.stl"/>
+        <origin xyz="0 0 -0.05" rpy="-1.5707 0 0"/>
+        <geometry>
+          <cylinder radius="0.03" length="0.03175"/>
         </geometry>
         <material name="light_grey">
@@ -113,7 +113,7 @@
       </inertial>
       <visual>
-        <origin xyz="0 0 0" rpy="-1.5707 0 1.5707"/>
-        <geometry>
-          <mesh filename="package://arlobot_ros/meshes/28971-Caster-Wheel-Kit-v1.0_simplified.stl"/>
+        <origin xyz="0 0 -0.05" rpy="-1.5707 0 0"/>
+        <geometry>
+          <cylinder radius="0.03" length="0.03175"/>
         </geometry>
         <material name="light_grey">
