Commit message: Finish cleanup of URDF description files.

File: urdf-xacro-source/arlo.urdf.xacro (robot description, xacro)
@@ -20,5 +20,5 @@
     <link name="base_footprint">
       <visual>
-        <origin xyz="0 0 0" rpy="0 0 0"/>
+      <origin rpy="0 0 0" xyz="0 0 0"/>
         <geometry>
           <box size="0.001 0.001 0.001"/>
@@ -27,5 +27,5 @@
       </visual>
       <collision>
-        <origin xyz="0 0 0.017" rpy="0 0 0"/>
+      <origin rpy="0 0 0" xyz="0 0 0.017"/>
         <geometry>
           <box size="0.001 0.001 0.001"/>
@@ -41,5 +41,5 @@
       </inertial>
       <visual>
-        <origin xyz="0 0 0" rpy="0 0 0"/>
+      <origin rpy="0 0 0" xyz="0 0 0"/>
         <geometry>
           <cylinder length="0.0095" radius="0.2245"/>
@@ -48,5 +48,5 @@
       </visual>
       <collision>
-        <origin xyz="0 0 0" rpy="0 0 0"/>
+      <origin rpy="0 0 0" xyz="0 0 0"/>
         <geometry>
           <cylinder length="0.0095" radius="0.2245"/>
@@ -63,5 +63,5 @@
       </inertial>
       <visual>
-        <origin xyz="0 0 0" rpy="0 0 0"/>
+      <origin rpy="0 0 0" xyz="0 0 0"/>
         <geometry>
           <box size="0.1778 0.3366 0.0762"/>
@@ -70,5 +70,5 @@
       </visual>
       <collision>
-        <origin xyz="0 0 0" rpy="0 0 0"/>
+      <origin rpy="0 0 0" xyz="0 0 0"/>
         <geometry>
           <box size="0.1778 0.3366 0.0762"/>
@@ -77,5 +77,5 @@
     </link>
     <joint name="battery_box_joint" type="fixed">
-      <origin xyz="0 0 -0.04285" rpy="0 0 0"/>
+    <origin rpy="0 0 0" xyz="0 0 -0.04285"/>
       <parent link="base_link"/>
       <child link="battery_box"/>
@@ -90,7 +90,7 @@
       </inertial>
       <visual>
-        <origin xyz="0 0 -0.05" rpy="-1.5707 0 0"/>
-        <geometry>
-          <cylinder radius="0.03" length="0.03175"/>
+      <origin rpy="-1.5707 0 0" xyz="0 0 -0.05"/>
+        <geometry>
+        <cylinder length="0.03175" radius="0.03"/>
         </geometry>
         <material name="light_grey">
@@ -100,5 +100,5 @@
     </link>
     <joint name="front_caster_joint" type="fixed">
-      <origin xyz="0.18745 0 -0.00475" rpy="0 0 0"/>
+    <origin rpy="0 0 0" xyz="0.18745 0 -0.00475"/>
       <parent link="base_link"/>
       <child link="front_caster"/>
@@ -113,7 +113,7 @@
       </inertial>
       <visual>
-        <origin xyz="0 0 -0.05" rpy="-1.5707 0 0"/>
-        <geometry>
-          <cylinder radius="0.03" length="0.03175"/>
+      <origin rpy="-1.5707 0 0" xyz="0 0 -0.05"/>
+        <geometry>
+        <cylinder length="0.03175" radius="0.03"/>
         </geometry>
         <material name="light_grey">
@@ -123,10 +123,10 @@
     </link>
     <joint name="rear_caster_joint" type="fixed">
-      <origin xyz="-0.18745 0 -0.00475" rpy="0 0 0"/>
+    <origin rpy="0 0 0" xyz="-0.18745 0 -0.00475"/>
       <parent link="base_link"/>
       <child link="rear_caster"/>
     </joint>
     <joint name="base_footprint_joint" type="fixed">
-      <origin xyz="0 0 0.10125" rpy="0 0 0"/>
+    <origin rpy="0 0 0" xyz="0 0 0.10125"/>
       <parent link="base_footprint"/>
       <child link="base_link"/>
@@ -140,19 +140,19 @@
       </inertial>
       <visual>
-        <origin xyz="0 0 0" rpy="0 1.5707 1.5707"/>
-        <geometry>
-          <cylinder radius="0.00635" length="0.00635"/>
+      <origin rpy="0 1.5707 1.5707" xyz="0 0 0"/>
+        <geometry>
+        <cylinder length="0.00635" radius="0.00635"/>
         </geometry>
         <material name="light_grey"/>
       </visual>
       <collision>
-        <origin xyz="0 0 0" rpy="0 1.5707 1.5707"/>
-        <geometry>
-          <cylinder radius="0.00635" length="0.00635"/>
+      <origin rpy="0 1.5707 1.5707" xyz="0 0 0"/>
+        <geometry>
+        <cylinder length="0.00635" radius="0.00635"/>
         </geometry>
       </collision>
     </link>
     <joint name="left_axle_joint" type="fixed">
-      <origin xyz="0 0.171475 0.0178" rpy="0 0 0"/>
+    <origin rpy="0 0 0" xyz="0 0.171475 0.0178"/>
       <parent link="battery_box"/>
       <child link="left_axle_link"/>
@@ -167,19 +167,19 @@
       </inertial>
       <visual>
-        <origin xyz="0 0 0" rpy="0 1.5707 1.5707"/>
-        <geometry>
-          <cylinder radius="0.00635" length="0.00635"/>
+      <origin rpy="0 1.5707 1.5707" xyz="0 0 0"/>
+        <geometry>
+        <cylinder length="0.00635" radius="0.00635"/>
         </geometry>
         <material name="light_grey"/>
       </visual>
       <collision>
-        <origin xyz="0 0 0" rpy="0 1.5707 1.5707"/>
-        <geometry>
-          <cylinder radius="0.00635" length="0.00635"/>
+      <origin rpy="0 1.5707 1.5707" xyz="0 0 0"/>
+        <geometry>
+        <cylinder length="0.00635" radius="0.00635"/>
         </geometry>
       </collision>
     </link>
     <joint name="right_axle_joint" type="fixed">
-      <origin xyz="0 -0.171475 0.0178" rpy="0 0 0"/>
+    <origin rpy="0 0 0" xyz="0 -0.171475 0.0178"/>
       <parent link="battery_box"/>
       <child link="right_axle_link"/>
@@ -194,14 +194,14 @@
       </inertial>
       <visual>
-        <origin xyz="0 0 0" rpy="0 1.5707 1.5707"/>
-        <geometry>
-          <cylinder radius="0.0762" length="0.03175"/>
+      <origin rpy="0 1.5707 1.5707" xyz="0 0 0"/>
+        <geometry>
+        <cylinder length="0.03175" radius="0.0762"/>
         </geometry>
         <material name="black"/>
       </visual>
       <collision>
-        <origin xyz="0 0 0" rpy="0 1.5707 1.5707"/>
-        <geometry>
-          <cylinder radius="0.0762" length="0.03175"/>
+      <origin rpy="0 1.5707 1.5707" xyz="0 0 0"/>
+        <geometry>
+        <cylinder length="0.03175" radius="0.0762"/>
         </geometry>
       </collision>
@@ -210,5 +210,5 @@
     <!-- NOTE This may prevent gazebo from working with this model -->
     <joint name="left_wheel_joint" type="fixed">
-      <origin xyz="0 0.01905 0" rpy="0 0 0"/>
+    <origin rpy="0 0 0" xyz="0 0.01905 0"/>
       <parent link="left_axle_link"/>
       <child link="left_wheel_link"/>
@@ -223,14 +223,14 @@
       </inertial>
       <visual>
-        <origin xyz="0 0 0" rpy="0 1.5707 1.5707"/>
-        <geometry>
-          <cylinder radius="0.0762" length="0.03175"/>
+      <origin rpy="0 1.5707 1.5707" xyz="0 0 0"/>
+        <geometry>
+        <cylinder length="0.03175" radius="0.0762"/>
         </geometry>
         <material name="black"/>
       </visual>
       <collision>
-        <origin xyz="0 0 0" rpy="0 1.5707 1.5707"/>
-        <geometry>
-          <cylinder radius="0.0762" length="0.03175"/>
+      <origin rpy="0 1.5707 1.5707" xyz="0 0 0"/>
+        <geometry>
+        <cylinder length="0.03175" radius="0.0762"/>
         </geometry>
       </collision>
@@ -239,5 +239,5 @@
     <!-- NOTE This may prevent gazebo from working with this model -->
     <joint name="right_wheel_joint" type="fixed">
-      <origin xyz="0 -0.01905 0" rpy="0 0 0"/>
+    <origin rpy="0 0 0" xyz="0 -0.01905 0"/>
       <parent link="right_axle_link"/>
       <child link="right_wheel_link"/>
@@ -246,5 +246,5 @@
     <!-- This pretends to be in the center in order to aid in calculating degrees from multiple sensors on one fake laser scan -->
     <joint name="ping_array_joint" type="fixed">
-      <origin xyz="0 0 0.03695" rpy="0 0 0"/>
+    <origin rpy="0 0 0" xyz="0 0 0.03695"/>
       <parent link="base_link"/>
       <child link="ping_sensor_array"/>
@@ -265,5 +265,5 @@
     </link>
     <joint name="ir_array_joint" type="fixed">
-      <origin xyz="0 0 0.03695" rpy="0 0 0"/>
+    <origin rpy="0 0 0" xyz="0 0 0.03695"/>
       <parent link="base_link"/>
       <child link="ir_sensor_array"/>
@@ -287,5 +287,5 @@
       <!-- Minor adjustments based on lining up Scanse Sweep output with 3D Sensor output -->
       <!-- So if the 3D sensor is misaligned the Scanse Sweep is off by the same amount -->
-      <origin xyz="0.15 0.0 0.269107" rpy="0 0 3.13"/>
+    <origin rpy="0 0 3.13" xyz="0.15 0.0 0.269107"/>
       <parent link="base_link"/>
       <child link="scanse_sweep"/>
@@ -315,5 +315,5 @@
       <!-- Hence the r of 3.1 to rotate it half way around.  -->
       <!-- The height is set even with the top plate. It shouldn't matter really. -->
-      <origin xyz="0.125 0.0 0.269107" rpy="0.0 0.0 0.0"/>
+    <origin rpy="0.0 0.0 0.0" xyz="0.125 0.0 0.269107"/>
       <parent link="base_link"/>
       <child link="rplidar"/>
@@ -349,5 +349,5 @@
       </inertial>
       <visual>
-        <origin xyz=" 0 0 0 " rpy="0 0 0"/>
+      <origin rpy="0 0 0" xyz=" 0 0 0 "/>
         <geometry>
           <cylinder length="0.127" radius="0.00635"/>
@@ -358,5 +358,5 @@
       </visual>
       <collision>
-        <origin xyz="0.0 0.0 0.0" rpy="0 0 0"/>
+      <origin rpy="0 0 0" xyz="0.0 0.0 0.0"/>
         <geometry>
           <cylinder length="0.127" radius="0.00635"/>
@@ -404,5 +404,5 @@
                           z_loc="0.06825"/>
     <joint name="plate_1_joint" type="fixed">
-      <origin xyz="0 0 0.1365" rpy="0 0 0"/>
+    <origin rpy="0 0 0" xyz="0 0 0.1365"/>
       <parent link="plate_0_link"/>
       <child link="plate_1_link"/>
@@ -417,5 +417,5 @@
       </inertial>
       <visual>
-        <origin xyz=" 0 0 0 " rpy="0 0 0"/>
+      <origin rpy="0 0 0" xyz=" 0 0 0 "/>
         <geometry>
           <cylinder length="0.0095" radius="0.2245"/>
@@ -426,5 +426,5 @@
       </visual>
       <collision>
-        <origin xyz="0.0 0.0 0.0" rpy="0 0 0"/>
+      <origin rpy="0 0 0" xyz="0.0 0.0 0.0"/>
         <geometry>
           <cylinder length="0.0095" radius="0.2245"/>
