Commit message: And now the actual working URD file in repo.

File: arlobot_ros/arlobot.urdf (robot description, URDF)
Before this commit: robot arlobot_hardware, 0 links, 0 joints
Links:
- added link base_footprint; collision box size=0.001 0.001 0.001; visual box size=0.001 0.001 0.001
- added link base_link, mass 2; collision cylinder length=0.0095 radius=0.2245; visual cylinder length=0.0095 radius=0.2245
- added link battery_box, mass 0.001; collision box size=0.1778 0.3366 0.0762; visual box size=0.1778 0.3366 0.0762
- added link front_caster, mass 0.001; visual cylinder length=0.03175 radius=0.03
- added link ir_sensor_array, mass 0.001; visual box size=0.0174 0.06 0.0644
- added link left_axle_link, mass 0.01; collision cylinder length=0.00635 radius=0.00635; visual cylinder length=0.00635 radius=0.00635
- added link left_wheel_link, mass 0.01; collision cylinder length=0.03175 radius=0.0762; visual cylinder length=0.03175 radius=0.0762
- added link ping_sensor_array, mass 0.001; visual box size=0.0174 0.06 0.0644
- added link plate_0_link, mass 0.01; collision cylinder length=0.0095 radius=0.2245; visual cylinder length=0.0095 radius=0.2245
- added link plate_1_link, mass 0.01; collision cylinder length=0.0095 radius=0.2245; visual cylinder length=0.0095 radius=0.2245
- added link rear_caster, mass 0.001; visual cylinder length=0.03175 radius=0.03
- added link right_axle_link, mass 0.01; collision cylinder length=0.00635 radius=0.00635; visual cylinder length=0.00635 radius=0.00635
- added link right_wheel_link, mass 0.01; collision cylinder length=0.03175 radius=0.0762; visual cylinder length=0.03175 radius=0.0762
- added link rplidar, mass 0.001; visual box size=0.0 0.0 0.0
- added link scanse_sweep, mass 0.001; visual box size=0.0 0.0 0.0
- added link standoff_5in_0_link, mass 0.001; collision cylinder length=0.127 radius=0.00635; visual cylinder length=0.127 radius=0.00635
- added link standoff_5in_1_link, mass 0.001; collision cylinder length=0.127 radius=0.00635; visual cylinder length=0.127 radius=0.00635
- added link standoff_5in_2_link, mass 0.001; collision cylinder length=0.127 radius=0.00635; visual cylinder length=0.127 radius=0.00635
- added link standoff_5in_3_link, mass 0.001; collision cylinder length=0.127 radius=0.00635; visual cylinder length=0.127 radius=0.00635
- added link standoff_5in_4_link, mass 0.001; collision cylinder length=0.127 radius=0.00635; visual cylinder length=0.127 radius=0.00635
- added link standoff_5in_5_link, mass 0.001; collision cylinder length=0.127 radius=0.00635; visual cylinder length=0.127 radius=0.00635
- added link standoff_5in_6_link, mass 0.001; collision cylinder length=0.127 radius=0.00635; visual cylinder length=0.127 radius=0.00635
- added link standoff_5in_7_link, mass 0.001; collision cylinder length=0.127 radius=0.00635; visual cylinder length=0.127 radius=0.00635
Joints:
- added joint base_footprint_joint: type fixed, parent base_footprint, child base_link, origin xyz=0 0 0.10125 rpy=0 0 0
- added joint battery_box_joint: type fixed, parent base_link, child battery_box, origin xyz=0 0 -0.04285 rpy=0 0 0
- added joint front_caster_joint: type fixed, parent base_link, child front_caster, origin xyz=0.18745 0 -0.00475 rpy=0 0 0
- added joint ir_array_joint: type fixed, parent base_link, child ir_sensor_array, origin xyz=0 0 0.03695 rpy=0 0 0
- added joint left_axle_joint: type fixed, parent battery_box, child left_axle_link, origin xyz=0 0.171475 0.0178 rpy=0 0 0, axis 0 1 0
- added joint left_wheel_joint: type fixed, parent left_axle_link, child left_wheel_link, origin xyz=0 0.01905 0 rpy=0 0 0, axis 0 1 0
- added joint ping_array_joint: type fixed, parent base_link, child ping_sensor_array, origin xyz=0 0 0.03695 rpy=0 0 0
- added joint plate_0_joint: type fixed, parent base_link, child plate_0_link, origin xyz=0 0 0.1365 rpy=0 0 0
- added joint plate_1_joint: type fixed, parent plate_0_link, child plate_1_link, origin xyz=0 0 0.1365 rpy=0 0 0
- added joint rear_caster_joint: type fixed, parent base_link, child rear_caster, origin xyz=-0.18745 0 -0.00475 rpy=0 0 0
- added joint right_axle_joint: type fixed, parent battery_box, child right_axle_link, origin xyz=0 -0.171475 0.0178 rpy=0 0 0, axis 0 1 0
- added joint right_wheel_joint: type fixed, parent right_axle_link, child right_wheel_link, origin xyz=0 -0.01905 0 rpy=0 0 0, axis 0 1 0
- added joint rplidar_joint: type fixed, parent base_link, child rplidar, origin xyz=0.125 0.0 0.269107 rpy=0.0 0.0 0.0
- added joint scanse_sweep_joint: type fixed, parent base_link, child scanse_sweep, origin xyz=0.15 0.0 0.269107 rpy=0 0 3.13
- added joint standoff_5in_0_joint: type fixed, parent base_link, child standoff_5in_0_link, origin xyz=0.0676402 0.1314196 0.06825 rpy=0 0 0
- added joint standoff_5in_1_joint: type fixed, parent base_link, child standoff_5in_1_link, origin xyz=0.0676402 -0.1314196 0.06825 rpy=0 0 0
- added joint standoff_5in_2_joint: type fixed, parent base_link, child standoff_5in_2_link, origin xyz=-0.052832 -0.1314196 0.06825 rpy=0 0 0
- added joint standoff_5in_3_joint: type fixed, parent base_link, child standoff_5in_3_link, origin xyz=-0.052832 0.1314196 0.06825 rpy=0 0 0
- added joint standoff_5in_4_joint: type fixed, parent plate_0_link, child standoff_5in_4_link, origin xyz=0.0676402 0.1314196 0.06825 rpy=0 0 0
- added joint standoff_5in_5_joint: type fixed, parent plate_0_link, child standoff_5in_5_link, origin xyz=0.0676402 -0.1314196 0.06825 rpy=0 0 0
- added joint standoff_5in_6_joint: type fixed, parent plate_0_link, child standoff_5in_6_link, origin xyz=-0.052832 -0.1314196 0.06825 rpy=0 0 0
- added joint standoff_5in_7_joint: type fixed, parent plate_0_link, child standoff_5in_7_link, origin xyz=-0.052832 0.1314196 0.06825 rpy=0 0 0
